Commit message: Cambios urdf

File: db_description/urdf/duckiebot.xacro (robot description, xacro)
@@ -3,19 +3,19 @@
   <xacro:property name="wheel_diameter"  value="0.034"/>
   <xacro:property name="wheel_thickness" value="0.025"/>
-  <xacro:property name="wheel_offset_z"  value="0.01"/>
+  <xacro:property name="wheel_offset_z"  value="0.034"/>
   <xacro:property name="wheel_ori_x"     value="0.055"/>
   <xacro:property name="chassis_ori_z"  value="0.0605"/>
   <xacro:property name="chassis_size_x" value="0.175"/>
-  <xacro:property name="chassis_size_y" value="0.081"/>
+  <xacro:property name="chassis_size_y" value="0.11"/>
   <xacro:property name="chassis_size_z" value="0.027"/>
   <xacro:property name="laser_ori_x"  value="0.0275"/>
   <xacro:property name="imu_ori_x"  value="-0.095"/>
   <!-- Base link -->
-  <link name="base_link"/>
+  <link name="base_link"/>.
   <!-- Chassis -->
   <xacro:macro name="chassis">
   <link name="chassis">
     <visual>
-      <origin xyz="0 0 ${chassis_ori_z}" rpy="0 0 0"/>
+      <origin xyz="0 0 ${chassis_ori_z} " rpy="0 0 0"/>
       <geometry>
         <box size="${chassis_size_x} ${chassis_size_y} ${chassis_size_z}"/>
@@ -59,9 +59,9 @@
       </visual>
     </link>
-    <joint name="imu_joint" type="fixed">
-      <parent link="chassis"/>
-      <child link="imu"/>
-      <origin xyz="${imu_ori_x} -0.006 0.0015" rpy="0 0 0"/>
-    </joint>
+  <joint name="imu_joint" type="fixed">
+    <parent link="chassis"/>
+    <child link="imu"/>
+    <origin xyz="${imu_ori_x} -0.006 0.0605" rpy="0 0 0"/>
+  </joint>
   </xacro:macro>
   <xacro:imu/>
@@ -91,5 +91,5 @@
     <parent link="chassis"/>
     <child link="left_wheel"/>
-    <origin xyz="0.05 -0.0625 0.015" rpy="${-pi/2} 0 0"/>
+    <origin xyz="0.05 -0.0625 0.017" rpy="${-pi/2} 0 0"/>
     <axis xyz="0 0 1"/>
   </joint>
@@ -97,5 +97,5 @@
     <parent link="chassis"/>
     <child link="right_wheel"/>
-    <origin xyz="0.05 0.0625 0.015" rpy="${pi/2} 0 0"/>
+    <origin xyz="0.05 0.0625 0.017" rpy="${pi/2} 0 0"/>
     <axis xyz="0 0 1"/>
   </joint>

Commit message: modificado 22nov

File: db_description/urdf/duckiebot.xacro (robot description, xacro)
@@ -3,19 +3,19 @@
   <xacro:property name="wheel_diameter"  value="0.034"/>
   <xacro:property name="wheel_thickness" value="0.025"/>
-  <xacro:property name="wheel_offset_z"  value="0.01"/>
+  <xacro:property name="wheel_offset_z"  value="0.034"/>
   <xacro:property name="wheel_ori_x"     value="0.055"/>
   <xacro:property name="chassis_ori_z"  value="0.0605"/>
   <xacro:property name="chassis_size_x" value="0.175"/>
-  <xacro:property name="chassis_size_y" value="0.081"/>
+  <xacro:property name="chassis_size_y" value="0.11"/>
   <xacro:property name="chassis_size_z" value="0.027"/>
   <xacro:property name="laser_ori_x"  value="0.0275"/>
   <xacro:property name="imu_ori_x"  value="-0.095"/>
   <!-- Base link -->
-  <link name="base_link"/>
+  <link name="base_link"/>.
   <!-- Chassis -->
   <xacro:macro name="chassis">
   <link name="chassis">
     <visual>
-      <origin xyz="0 0 ${chassis_ori_z}" rpy="0 0 0"/>
+      <origin xyz="0 0 ${chassis_ori_z} " rpy="0 0 0"/>
       <geometry>
         <box size="${chassis_size_x} ${chassis_size_y} ${chassis_size_z}"/>
@@ -59,9 +59,9 @@
       </visual>
     </link>
-    <joint name="imu_joint" type="fixed">
-      <parent link="chassis"/>
-      <child link="imu"/>
-      <origin xyz="${imu_ori_x} -0.006 0.0015" rpy="0 0 0"/>
-    </joint>
+  <joint name="imu_joint" type="fixed">
+    <parent link="chassis"/>
+    <child link="imu"/>
+    <origin xyz="${imu_ori_x} -0.006 0.059" rpy="0 0 0"/>
+  </joint>
   </xacro:macro>
   <xacro:imu/>
@@ -91,5 +91,5 @@
     <parent link="chassis"/>
     <child link="left_wheel"/>
-    <origin xyz="0.05 -0.0625 0.015" rpy="${-pi/2} 0 0"/>
+    <origin xyz="0.05 -0.0625 0.017" rpy="${-pi/2} 0 0"/>
     <axis xyz="0 0 1"/>
   </joint>
@@ -97,5 +97,5 @@
     <parent link="chassis"/>
     <child link="right_wheel"/>
-    <origin xyz="0.05 0.0625 0.015" rpy="${pi/2} 0 0"/>
+    <origin xyz="0.05 0.0625 0.017" rpy="${pi/2} 0 0"/>
     <axis xyz="0 0 1"/>
   </joint>

Commit message: Final final ahora si que si gol de oro

File: db_description/urdf/duckiebot.xacro (robot description, xacro)
@@ -62,9 +62,5 @@
     <parent link="chassis"/>
     <child link="imu"/>
-<<<<<<< HEAD
-    <origin xyz="${imu_ori_x} -0.006 0.0605" rpy="0 0 0"/>
-=======
     <origin xyz="${imu_ori_x} -0.006 0.059" rpy="0 0 0"/>
->>>>>>> dff2cbfa8f1e050f65681102396b1126979ddf8e
   </joint>
   </xacro:macro>
